File: Blinky_5.0/GettingToBlinky5.0.kicad_pcb (KiCad board)
At the start: 2 copper layers, 34 x 30 mm, 7 parts

Commit message: Just resetting I messed up somewhere?
Parts:
- removed BT1: CR2032, Library:Untitled
- removed C1: 1u, Capacitor_SMD:C_0805_2012Metric
- removed D1: LED, LED_SMD:LED_0805_2012Metric
- removed R1: 1K, Resistor_SMD:R_0805_2012Metric
- removed R2: 470k, Resistor_SMD:R_0805_2012Metric
- removed R3: 1k, Resistor_SMD:R_0805_2012Metric
- removed U-2: ~, Package_SO:SO-8_3.9x4.9mm_P1.27mm
Routing:
- net Net-(U-2-THR): track 15.2 -> 0.00 mm
- net /Vdd: track 8.64 -> 0.00 mm, vias 2 -> 0
- net Net-(U-2-DIS): track 5.82 -> 0.00 mm
- net GND: track 5.73 -> 0.00 mm, vias 3 -> 0
- net Net-(U-2-OUT): track 4.03 -> 0.00 mm
- net Net-(D1-A): track 2.70 -> 0.00 mm
- removed copper zone on F.Cu, net /Vdd
- removed copper zone on B.Cu, net GND
Other:
- board outline removed

Commit message: No errors generating gerber
Parts:
- added BT1: CR2032, Library:C-Battery, F.Cu at (140.2, 107.4)
- added C1: 1u, Capacitor_SMD:C_0805_2012Metric, F.Cu at (134.7, 109.8)
- added D1: LED, LED_SMD:LED_0805_2012Metric, F.Cu at (134.7, 117.8)
- added R1: 1K, Resistor_SMD:R_0805_2012Metric, F.Cu at (147.6, 109.6)
- added R2: 470k, Resistor_SMD:R_0805_2012Metric, F.Cu at (147.6, 113.6)
- added R3: 1k, Resistor_SMD:R_0805_2012Metric, F.Cu at (134.7, 113.6)
- added U-2: ~, Package_SO:SO-8_3.9x4.9mm_P1.27mm, F.Cu at (141.2, 111.4)
Routing:
- net /THR: track 0.00 -> 14.5 mm
- net /Vdd: track 0.00 -> 12.8 mm, vias 0 -> 2
- net /DIS: track 0.00 -> 6.07 mm
- net GND: track 0.00 -> 5.18 mm, vias 0 -> 3
- net Net-(U-2-OUT): track 0.00 -> 4.23 mm
- net Net-(D1-A): track 0.00 -> 2.33 mm
- added copper zone on F.Cu, net /Vdd
- added copper zone on B.Cu, net GND
Other:
- board outline added: 40 x 40 mm
- board text added: "Blinky LED"
- board text added: "Made by: Gabe"
