File: Blinky_5.0/GettingToBlinky5.0.kicad_pcb (KiCad board)
At the start: 2 copper layers, 40 x 40 mm, 7 parts

Commit message: Forgot to hit save
Parts:
- BT1: moved to B.Cu
- moved BT1 1.80 mm to (142.0, 107.3), turned to 180 degrees
Changed lines of the file:
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@@
 		)
-	)
-	(footprint "Library:C-Battery"
-		(layer "F.Cu")
-		(at 140.2 107.4)
-		(property "Reference" "BT1"
-			(at 1.1 6.8 0)
-			(unlocked yes)
-			(layer "F.SilkS")
-			(effects
-				(font
-					(size 1 1)
-					(thickness 0.1)
-				)
-			)
-		)
-		(property "Value" "CR2032"
-			(at 1.1 0.9 0)
-			(unlocked yes)
-			(layer "F.Fab")
-			(effects
-				(font
-					(size 1 1)
-					(thickness 0.15)
-				)
-			)
-		)
-		(property "Datasheet" ""
-			(at 0 0 0)
-			(unlocked yes)
-			(layer "F.Fab")
-			(hide yes)
-			(effects
-				(font
-					(size 1 1)
-					(thickness 0.15)
-				)
-			)
-		)
-		(property "Description" "Single-cell battery"
-			(at 0 0 0)
-			(unlocked yes)
-			(layer "F.Fab")
-			(hide yes)
-			(effects
-				(font
-					(size 1 1)
-					(thickness 0.15)
-				)
-			)
-		)
-		(sheetname "/")
-		(sheetfile "GettingToBlinky5.0.kicad_sch")
-		(attr smd)
-		(fp_line
-			(start -9 -6.5)
-			(end 11 -6.5)
-			(stroke
-				(width 0.1)
-				(type default)
-			)
-			(layer "F.SilkS")
-		)
-		(fp_line
-			(start -9 14.5)
-			(end -9 -6.5)
-			(stroke
-				(width 0.1)
-				(type default)
-			)
-			(layer "F.SilkS")
-		)
-		(fp_line
-			(start -9 14.5)
-			(end 11 14.5)
-			(stroke
-				(width 0.1)
-				(type default)
-			)
-			(layer "F.SilkS")
-		)
-		(fp_line
-			(start 11 -6.5)
-			(end 11 14.5)
-			(stroke
-				(width 0.1)
-				(type default)
-			)
-			(layer "F.SilkS")
-		)
-		(fp_line
-			(start -16 21)
-			(end -16 -13)
-			(stroke
-				(width 0.05)
-				(type default)
-			)
-			(layer "F.CrtYd")
-		)
-		(fp_line
-			(start 18 -13)
-			(end -16 -13)
-			(stroke
-				(width 0.05)
-				(type default)
-			)
-			(layer "F.CrtYd")
-		)
-		(fp_line
-			(start 18 21)
-			(end -16 21)
-			(stroke
-				(width 0.05)
-				(type default)
-			)
-			(layer "F.CrtYd")
-		)
-		(fp_line
-			(start 18 21)
-			(end 18 -13)
-			(stroke
-				(width 0.05)
-				(type default)
-			)
-			(layer "F.CrtYd")
-		)
-		(fp_text user "${REFERENCE}"
-			(at 1 8.3 0)
-			(unlocked yes)
-			(layer "F.Fab")
-			(effects
-				(font
-					(size 1 1)
-					(thickness 0.15)
-				)
-			)
-		)
-		(pad "1" smd rect
-			(at -11.8 4)
-			(size 5.5 5.5)
-			(layers "F.Cu" "F.Mask" "F.Paste")
-			(net 5 "/Vdd")
-			(pinfunction "+")
-			(pintype "passive")
-			(thermal_bridge_angle 45)
-		)
-		(pad "1" smd rect
-			(at 13.8 4)
-			(size 5.5 5.5)
-			(layers "F.Cu" "F.Mask" "F.Paste")
-			(net 5 "/Vdd")
-			(pinfunction "+")
-			(pintype "passive")
-			(thermal_bridge_angle 45)
-		)
-		(pad "2" smd rect
-			(at 1 4)
-			(size 4 4)
-			(layers "F.Cu" "F.Mask" "F.Paste")
-			(net 1 "GND")
-			(pinfunction "-")
-			(pintype "passive")
-			(thermal_bridge_angle 45)
-		)
-		(embedded_fonts no)
 	)
 	(footprint "Resistor_SMD:R_0805_2012Metric"
@@
 		)
 	)
+	(footprint "Library:C-Battery"
+		(layer "B.Cu")
+		(at 142 107.3 180)
+		(property "Reference" "BT1"
+			(at 1.1 -6.8 0)
+			(unlocked yes)
+			(layer "B.SilkS")
+			(effects
+				(font
+					(size 1 1)
+					(thickness 0.1)
+				)
+				(justify mirror)
+			)
+		)
+		(property "Value" "CR2032"
+			(at 1.1 -0.9 0)
+			(unlocked yes)
+			(layer "B.Fab")
+			(effects
+				(font
+					(size 1 1)
+					(thickness 0.15)
+				)
+				(justify mirror)
+			)
+		)
+		(property "Datasheet" ""
+			(at 0 0 0)
+			(unlocked yes)
+			(layer "B.Fab")
+			(hide yes)
+			(effects
+				(font
+					(size 1 1)
+					(thickness 0.15)
+				)
+				(justify mirror)
+			)
+		)
+		(property "Description" "Single-cell battery"
+			(at 0 0 0)
+			(unlocked yes)
+			(layer "B.Fab")
+			(hide yes)
+			(effects
+				(font
+					(size 1 1)
+					(thickness 0.15)
+				)
+				(justify mirror)
+			)
+		)
+		(sheetname "/")
+		(sheetfile "GettingToBlinky5.0.kicad_sch")
+		(attr smd)
+		(fp_line
+			(start 11 6.5)
+			(end 11 -14.5)
+			(stroke
+				(width 0.1)
+				(type default)
+			)
+			(layer "B.SilkS")
+		)
+		(fp_line
+			(start -9 6.5)
+			(end 11 6.5)
+			(stroke
+				(width 0.1)
+				(type default)
+			)
+			(layer "B.SilkS")
+		)
+		(fp_line
+			(start -9 -14.5)
+			(end 11 -14.5)
+			(stroke
+				(width 0.1)
+				(type default)
+			)
+			(layer "B.SilkS")
+		)
+		(fp_line
+			(start -9 -14.5)
+			(end -9 6.5)
+			(stroke
+				(width 0.1)
+				(type default)
+			)
+			(layer "B.SilkS")
+		)
+		(fp_line
+			(start 18 13)
+			(end -16 13)
+			(stroke
+				(width 0.05)
+				(type default)
+			)
+			(layer "B.CrtYd")
+		)
+		(fp_line
+			(start 18 -21)
+			(end 18 13)
+			(stroke
+				(width 0.05)
+				(type default)
+			)
+			(layer "B.CrtYd")
+		)
+		(fp_line
+			(start 18 -21)
+			(end -16 -21)
+			(stroke
+				(width 0.05)
+				(type default)
+			)
+			(layer "B.CrtYd")
+		)
+		(fp_line
+			(start -16 -21)
+			(end -16 13)
+			(stroke
+				(width 0.05)
+				(type default)
+			)
+			(layer "B.CrtYd")
+		)
+		(fp_text user "${REFERENCE}"
+			(at 1 -8.3 0)
+			(unlocked yes)
+			(layer "B.Fab")
+			(effects
+				(font
+					(size 1 1)
+					(thickness 0.15)
+				)
+				(justify mirror)
+			)
+		)
+		(pad "1" smd rect
+			(at -11.8 -4 180)
+			(size 5.5 5.5)
+			(layers "B.Cu" "B.Mask" "B.Paste")
+			(net 5 "/Vdd")
+			(pinfunction "+")
+			(pintype "passive")
+			(thermal_bridge_angle 45)
+		)
+		(pad "1" smd rect
+			(at 13.8 -4 180)
+			(size 5.5 5.5)
+			(layers "B.Cu" "B.Mask" "B.Paste")
+			(net 5 "/Vdd")
+			(pinfunction "+")
+			(pintype "passive")
+			(thermal_bridge_angle 45)
+		)
+		(pad "2" smd rect
+			(at 1 -4 180)
+			(size 4 4)
+			(layers "B.Cu" "B.Mask" "B.Paste")
+			(net 1 "GND")
+			(pinfunction "-")
+			(pintype "passive")
+			(thermal_bridge_angle 45)
+		)
+		(embedded_fonts no)
+	)
 	(gr_line
 		(start 161 92)
@@
 	)
 	(gr_text "Made by: \nGabe"
-		(at 143.7 126.2 0)
+		(at 143.7 127.4 0)
 		(layer "F.Cu" knockout)
 		(effects
@@
 	)
 	(gr_text "Blinky LED"
-		(at 135 101 0)
+		(at 135 100 0)
 		(layer "F.SilkS")
 		(effects
