File: Blinky_5.0/GettingToBlinky5.0.kicad_sch (KiCad schematic)
At the start: 0 parts

Commit message: Added Schematic
Parts:
- added BT1: CR2032, symbol Device:Battery_Cell
- added C1: 1u, symbol Device:C
- added D1: LED, symbol Device:LED
- added R1: 1K, symbol Device:R
- added R2: 470k, symbol Device:R
- added R3: 1k, symbol Device:R
- added U-2: ~, symbol GTB5kicad_sym:7555
Connections:
- new net: C1.1, R2.2, U-2.2 (~TRIG), U-2.6 (THR)
- new net: R3.1, U-2.3 (OUT)
- new net: BT1.1 (+), R1.1, U-2.4 (~RST), U-2.8 (VDD)
- new net: R1.2, R2.1, U-2.7 (DIS)
- new net: D1.2 (A), R3.2
- new net GND: BT1.2 (-), C1.2, D1.1 (K), U-2.1 (GND)
- no-connect marks 0 -> 1

Commit message: Made Custon Footprint
Parts:
- BT1: footprint (none) -> Library:Untitled
- C1: footprint (none) -> Capacitor_SMD:C_0805_2012Metric
- D1: footprint (none) -> LED_SMD:LED_0805_2012Metric
- R1, R2, R3: footprint (none) -> Resistor_SMD:R_0805_2012Metric
- U-2: footprint (none) -> Package_SO:SO-8_3.9x4.9mm_P1.27mm
Changed lines of the file:
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@@
 			)
 		)
-		(property "Footprint" ""
+		(property "Footprint" "Package_SO:SO-8_3.9x4.9mm_P1.27mm"
 			(at 149.86 115.57 0)
 			(effects
@@
 			)
 		)
-		(property "Footprint" ""
+		(property "Footprint" "Resistor_SMD:R_0805_2012Metric"
 			(at 170.942 101.6 90)
 			(effects
@@
 			)
 		)
-		(property "Footprint" ""
+		(property "Footprint" "Resistor_SMD:R_0805_2012Metric"
 			(at 117.602 96.52 90)
 			(effects
@@
 			)
 		)
-		(property "Footprint" ""
+		(property "Footprint" "LED_SMD:LED_0805_2012Metric"
 			(at 172.72 116.84 0)
 			(effects
@@
 			)
 		)
-		(property "Footprint" ""
+		(property "Footprint" "Resistor_SMD:R_0805_2012Metric"
 			(at 117.602 74.93 90)
 			(effects
@@
 			)
 		)
-		(property "Footprint" ""
+		(property "Footprint" "Library:Untitled"
 			(at 91.44 94.996 90)
 			(effects
@@
 			)
 		)
-		(property "Footprint" ""
+		(property "Footprint" "Capacitor_SMD:C_0805_2012Metric"
 			(at 120.3452 119.38 0)
 			(effects

Commit message: PCB Edited
Connections:
- net Vdd: now reaches BT1.1 (+), R1.1, U-2.4 (~RST), U-2.8 (VDD)
Changed lines of the file:
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@@
+		)
+	)
+	(label "Vdd"
+		(at 140.97 66.04 0)
+		(effects
+			(font
+				(size 1.27 1.27)
+			)
+			(justify left bottom)
 		)
 	)

Commit message: No errors generating gerber
Parts:
- BT1: footprint Library:Untitled -> Library:C-Battery
Connections:
- net THR: now reaches C1.1, R2.2, U-2.2 (~TRIG), U-2.6 (THR)
- net DIS: now reaches R1.2, R2.1, U-2.7 (DIS)
Changed lines of the file:
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@@
 	(paper "A4")
+	(junction
+		(at 128.27 127)
+		(diameter 0)
+		(color 0 0 0 0)
+	)
 	(junction
 		(at 130.81 105.41)
@@
 	(wire
 		(pts
-			(xy 148.59 127) (xy 119.38 127)
+			(xy 148.59 127) (xy 128.27 127)
 		)
 		(stroke
@@
 	(wire
 		(pts
+			(xy 128.27 127) (xy 119.38 127)
+		)
+		(stroke
+			(width 0)
+			(type default)
+		)
+	)
+	(wire
+		(pts
 			(xy 138.43 93.98) (xy 130.81 93.98)
 		)
@@
 			(width 0)
 			(type default)
+		)
+	)
+	(label "DIS"
+		(at 129.54 90.17 0)
+		(effects
+			(font
+				(size 1.27 1.27)
+			)
+			(justify left bottom)
+		)
+	)
+	(label "THR"
+		(at 132.08 93.98 0)
+		(effects
+			(font
+				(size 1.27 1.27)
+			)
+			(justify left bottom)
 		)
 	)
@@
 	)
 	(symbol
+		(lib_id "power:PWR_FLAG")
+		(at 128.27 127 0)
+		(unit 1)
+		(exclude_from_sim no)
+		(in_bom yes)
+		(on_board yes)
+		(dnp no)
+		(fields_autoplaced yes)
+		(property "Reference" "#FLG02"
+			(at 128.27 125.095 0)
+			(effects
+				(font
+					(size 1.27 1.27)
+				)
+				(hide yes)
+			)
+		)
+		(property "Value" "PWR_FLAG"
+			(at 128.27 121.92 0)
+			(effects
+				(font
+					(size 1.27 1.27)
+				)
+			)
+		)
+		(property "Footprint" ""
+			(at 128.27 127 0)
+			(effects
+				(font
+					(size 1.27 1.27)
+				)
+				(hide yes)
+			)
+		)
+		(property "Datasheet" "~"
+			(at 128.27 127 0)
+			(effects
+				(font
+					(size 1.27 1.27)
+				)
+				(hide yes)
+			)
+		)
+		(property "Description" "Special symbol for telling ERC where power comes from"
+			(at 128.27 127 0)
+			(effects
+				(font
+					(size 1.27 1.27)
+				)
+				(hide yes)
+			)
+		)
+		(pin "1"
+		)
+		(instances
+			(project "GettingToBlinky5.0"
+				(path "/7f07159f-9863-4848-a0e7-b5aa6dd12754"
+					(reference "#FLG02")
+					(unit 1)
+				)
+			)
+		)
+	)
+	(symbol
 		(lib_id "Device:R")
 		(at 119.38 96.52 0)
@@
 			)
 		)
-		(property "Footprint" "Library:Untitled"
+		(property "Footprint" "Library:C-Battery"
 			(at 91.44 94.996 90)
 			(effects
