File: colorful_LED/design/design.kicad_pcb (KiCad board)
At the start: 2 copper layers, 37 parts, among them J1 USB_B, SW1 SW_Push, SW2 SW_Wuerth_450301014042, U1 ATmega32U4-A, Y1 8MHz

Commit message: traces etched
Parts:
- C6, C7, C8, D2, L1, R5, R6, U2: moved to B.Cu
- moved DS1 67.1 mm to (163.6, 109.8), turned to 90 degrees
- moved R8 57.8 mm to (113.1, 109.2), turned to 180 degrees
- moved R7 57.7 mm to (113.0, 105.0), turned to 180 degrees
- moved R9 56.7 mm to (113.1, 107.2), turned to 180 degrees
- moved D5 56.1 mm to (102.4, 107.5)
- moved R11 49.3 mm to (153.6, 110.7), turned to 90 degrees
- moved R10 45.8 mm to (153.6, 106.5), turned to 90 degrees
- moved L1 36.1 mm to (161.1, 88.0), turned to 180 degrees
- moved BT1 34.4 mm to (152.1, 84.2)
- moved U2 33.1 mm to (159.2, 85.2), turned to 180 degrees
- moved R1 31.2 mm to (119.2, 84.5), turned to -90 degrees
- moved C4 30.6 mm to (143.3, 107.8), turned to -90 degrees
- moved C7 29.6 mm to (157.9, 89.0), turned to 90 degrees
- moved D2 29.0 mm to (163.1, 94.4)
- moved RV1 28.8 mm to (128.5, 91.4)
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Routing:
- net VBOOST: track 0.00 -> 86.9 mm
- net VBUS: track 0.00 -> 48.0 mm
- net UGND: track 0.00 -> 42.0 mm
- net SCL: track 0.00 -> 32.1 mm
- net SDA: track 0.00 -> 31.7 mm
- net D+: track 0.00 -> 28.6 mm
- net Net-(J1-D-): track 0.00 -> 26.7 mm
- net D-: track 0.00 -> 24.4 mm
- net DGND: track 0.00 -> 23.5 mm, vias 0 -> 13
- net Net-(J1-Shield): track 0.00 -> 21.8 mm, vias 0 -> 1
- net Net-(D2-A): track 0.00 -> 19.4 mm, vias 0 -> 2
- net Net-(U2-FB): track 0.00 -> 17.3 mm
- net R_LEG: track 0.00 -> 16.8 mm
- net Net-(J1-D+): track 0.00 -> 16.6 mm
- net G_LEG: track 0.00 -> 16.1 mm
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- added copper zone on In2.Cu, net AGND
- added copper zone on In1.Cu, net AVCC
- removed copper zone on B.Cu, net AVCC
Other:
- board outline added: 66.5 x 60 mm
- copper layers 2 -> 4
- board text added: "BATT"
- board text added: "USB"
